File: MESC_IMS_ESC.kicad_pcb (KiCad board)
At the start: 4 copper layers, 0 parts

Commit message: Assigned all footprints
Began initial placement
Parts:
- added C1: 100pF, Capacitor_SMD:C_0402_1005Metric, F.Cu at (207.0, 85.0)
- added C10: 100nF, Capacitor_SMD:C_0402_1005Metric, F.Cu at (194.5, 89.5)
- added C11: 100nF, Capacitor_SMD:C_0402_1005Metric, F.Cu at (194.5, 82.0)
- added C12: 100nF, Capacitor_SMD:C_0402_1005Metric, F.Cu at (194.5, 87.0)
- added C13: 100nF, Capacitor_SMD:C_0402_1005Metric, F.Cu at (194.5, 84.5)
- added C14: 1uF, Capacitor_SMD:C_0402_1005Metric, F.Cu at (194.5, 92.0)
- added C15: 1uF, Capacitor_SMD:C_0402_1005Metric, F.Cu at (199.5, 129.5)
- added C16: 100nF, Capacitor_SMD:C_0805_2012Metric, F.Cu at (119.5, 144.0)
- added C17: 1uF, Capacitor_SMD:C_1206_3216Metric, F.Cu at (116.0, 144.0)
- added C18: 1uF, Capacitor_SMD:C_1206_3216Metric, F.Cu at (112.5, 144.0)
- added C19: 1uF 16V, Capacitor_SMD:C_0603_1608Metric, F.Cu at (139.2, 90.5)
- added C2: 100pF, Capacitor_SMD:C_0402_1005Metric, F.Cu at (207.0, 83.0)
- added C20: 1uF 16V, Capacitor_SMD:C_0603_1608Metric, F.Cu at (114.7, 128.5)
- added C21: 10nF 25V, Capacitor_SMD:C_0603_1608Metric, F.Cu at (111.7, 128.5)
- added C22: 4.7uF 6.3V, Capacitor_SMD:C_0805_2012Metric, F.Cu at (138.9, 84.0)
- added C23: 100nF, Capacitor_SMD:C_0402_1005Metric, F.Cu at (103.5, 116.5)
- added C24: 3.3nF, Capacitor_SMD:C_0402_1005Metric, F.Cu at (104.5, 114.0)
- added C25: 10uF, Capacitor_SMD:C_1206_3216Metric, F.Cu at (115.5, 106.0)
- added C26: 10uF, Capacitor_SMD:C_1206_3216Metric, F.Cu at (109.5, 106.0)
- added C27: 10uF, Capacitor_SMD:C_1206_3216Metric, F.Cu at (115.5, 102.0)
- added C28: 10uF, Capacitor_SMD:C_1206_3216Metric, F.Cu at (109.5, 102.0)
- added C29: 100pF, Capacitor_SMD:C_0402_1005Metric, F.Cu at (197.0, 101.0)
- added C3: 100pF, Capacitor_SMD:C_0402_1005Metric, F.Cu at (154.0, 96.5)
- added C30: 100pF, Capacitor_SMD:C_0402_1005Metric, F.Cu at (194.0, 101.0)
- added C31: C, Capacitor_SMD:C_0603_1608Metric, F.Cu at (188.5, 100.7)
- added C32: 100nF, Capacitor_SMD:C_0402_1005Metric, F.Cu at (192.5, 101.5)
- added C34: 100nF, Capacitor_SMD:C_0402_1005Metric, F.Cu at (184.0, 120.5)
- added C35: 1uF 50V, Capacitor_SMD:C_0805_2012Metric, F.Cu at (194.6, 116.0)
- added C36: 1uF 50V, Capacitor_SMD:C_0805_2012Metric, F.Cu at (188.0, 116.5)
- added C37: 100pF, Capacitor_SMD:C_0402_1005Metric, F.Cu at (201.5, 124.0)
- added C38: 100pF, Capacitor_SMD:C_0402_1005Metric, F.Cu at (168.5, 104.0)
- added C39: 100pF, Capacitor_SMD:C_0402_1005Metric, F.Cu at (165.5, 104.0)
- added C4: 100pF, Capacitor_SMD:C_0402_1005Metric, F.Cu at (207.0, 81.0)
- added C40: C, Capacitor_SMD:C_0603_1608Metric, F.Cu at (162.0, 103.2)
- added C41: 100nF, Capacitor_SMD:C_0402_1005Metric, F.Cu at (172.5, 127.0)
- added C43: 100nF, Capacitor_SMD:C_0402_1005Metric, F.Cu at (154.0, 120.0)
- added C44: 1uF 50V, Capacitor_SMD:C_0805_2012Metric, F.Cu at (166.1, 118.5)
- added C45: 1uF 50V, Capacitor_SMD:C_0805_2012Metric, F.Cu at (159.6, 118.5)
- added C46: 100pF, Capacitor_SMD:C_0402_1005Metric, F.Cu at (170.0, 125.0)
- added C47: 100pF, Capacitor_SMD:C_0402_1005Metric, F.Cu at (141.5, 104.5)
- added C48: 100pF, Capacitor_SMD:C_0402_1005Metric, F.Cu at (138.5, 104.5)
- added C49: C, Capacitor_SMD:C_0603_1608Metric, F.Cu at (134.5, 103.7)
- added C5: 100nF, Capacitor_SMD:C_0402_1005Metric, F.Cu at (152.0, 76.5)
- added C50: 100nF, Capacitor_SMD:C_0402_1005Metric, F.Cu at (137.0, 105.0)
- added C52: 100nF, Capacitor_SMD:C_0402_1005Metric, F.Cu at (128.0, 121.0)
- added C53: 1uF 50V, Capacitor_SMD:C_0805_2012Metric, F.Cu at (139.5, 120.0)
- added C54: 1uF 50V, Capacitor_SMD:C_0805_2012Metric, F.Cu at (133.0, 120.0)
- added C55: 100pF, Capacitor_SMD:C_0402_1005Metric, F.Cu at (143.0, 128.5)
- added C6: 100nF, Capacitor_SMD:C_0402_1005Metric, F.Cu at (124.5, 86.0)
- added C7: 100nF, Capacitor_SMD:C_0402_1005Metric, F.Cu at (177.0, 82.0)
- added C8: 100nF, Capacitor_SMD:C_0402_1005Metric, F.Cu at (194.5, 79.3)
- added C9: 100nF, Capacitor_SMD:C_0402_1005Metric, F.Cu at (119.5, 100.5)
- added D1: NSR1020MW2T1G, Diode_SMD:D_SOD-323, F.Cu at (183.5, 78.0)
- added D10: NSR1020MW2T1G, Diode_SMD:D_SOD-323, F.Cu at (199.0, 120.5)
- added D11: D_Schottky_Small, Diode_SMD:D_SMB, F.Cu at (171.0, 117.5)
- added D12: MMSZ18T1G, Diode_SMD:D_SOD-123, F.Cu at (164.0, 129.5)
- added D13: MMSZ18T1G, Diode_SMD:D_SOD-123, F.Cu at (159.0, 129.5)
- added D14: NSR1020MW2T1G, Diode_SMD:D_SOD-323, F.Cu at (172.5, 124.5)
- added D15: D_Schottky_Small, Diode_SMD:D_SMB, F.Cu at (144.5, 118.5)
- added D16: MMSZ18T1G, Diode_SMD:D_SOD-123, F.Cu at (138.5, 129.0)
- added D17: MMSZ18T1G, Diode_SMD:D_SOD-123, F.Cu at (133.3, 129.0)
- added D18: NSR1020MW2T1G, Diode_SMD:D_SOD-323, F.Cu at (144.9, 124.5)
- added D2: NSR1020MW2T1G, Diode_SMD:D_SOD-323, F.Cu at (152.5, 94.0)
- added D3: NSR1020MW2T1G, Diode_SMD:D_SOD-323, F.Cu at (121.0, 85.5)
- added D4: NSR1020MW2T1G, Diode_SMD:D_SOD-323, F.Cu at (116.0, 102.5)
- added D5: KP-1608MGC, Diode_SMD:D_0603_1608Metric, F.Cu at (138.0, 81.0)
- added D6: MBR130, Diode_SMD:D_SOD-123, F.Cu at (123.0, 118.5)
- added D7: D_Schottky_Small, Diode_SMD:D_SMB, F.Cu at (200.0, 113.5)
- added D8: MMSZ18T1G, Diode_SMD:D_SOD-123, F.Cu at (194.0, 126.5)
- added D9: MMSZ18T1G, Diode_SMD:D_SOD-123, F.Cu at (189.0, 126.5)
- added J1: Conn_01x08_Female, Connector_PinSocket_2.54mm:PinSocket_1x08_P2.54mm_Horizontal, F.Cu at (183.0, 132.5)
- added J2: Conn_01x08_Female, Connector_PinSocket_2.54mm:PinSocket_1x08_P2.54mm_Horizontal, F.Cu at (152.5, 133.0)
- added J3: Conn_01x08_Female, Connector_PinSocket_2.54mm:PinSocket_1x08_P2.54mm_Horizontal, F.Cu at (127.0, 133.5)
- added J4: Conn_01x06_Male, Connector_JST:JST_PH_B6B-PH-K_1x06_P2.00mm_Vertical, F.Cu at (215.5, 79.0)
- added J5: Conn_ARM_JTAG_SWD_10, Connector_PinHeader_1.27mm:PinHeader_2x05_P1.27mm_Vertical, F.Cu at (178.5, 77.0)
- added J6: USB_C_Receptacle_USB2.0, Connector_USB:USB_C_Receptacle_Palconn_UTC16-G, F.Cu at (105.0, 84.0)
- added J7: Conn_01x03_Male, Connector_PinHeader_2.54mm:PinHeader_1x03_P2.54mm_Vertical, F.Cu at (148.0, 91.5)
- added J8: Conn_01x04_Male, Connector_PinHeader_2.54mm:PinHeader_1x04_P2.54mm_Vertical, F.Cu at (215.5, 104.0)
- added J9: Conn_01x08_Male, Connector_JST:JST_PH_B8B-PH-K_1x08_P2.00mm_Vertical, F.Cu at (118.5, 78.5)
- added JP1: Jumper_NC_Small, Jumper:SolderJumper-2_P1.3mm_Bridged_RoundedPad1.0x1.5mm, F.Cu at (176.0, 99.0)
- added L1: SRF1260-101M, Inductor_SMD:L_Bourns_SRF1260, F.Cu at (113.5, 117.5)
- added R1: 1k5, Resistor_SMD:R_0402_1005Metric, F.Cu at (210.0, 86.0)
- added R10: 4k7, Resistor_SMD:R_0402_1005Metric, F.Cu at (210.0, 82.5)
- added R11: 1k5, Resistor_SMD:R_0402_1005Metric, F.Cu at (210.0, 80.0)
- added R12: 100R, Resistor_SMD:R_0402_1005Metric, F.Cu at (152.0, 96.5)
- added R13: 4k7, Resistor_SMD:R_0402_1005Metric, F.Cu at (210.0, 81.0)
- added R14: 1k5, Resistor_SMD:R_0402_1005Metric, F.Cu at (211.5, 96.0)
- added R15: 1k, Resistor_SMD:R_0402_1005Metric, F.Cu at (149.0, 79.0)
- added R16: 1k5, Resistor_SMD:R_0402_1005Metric, F.Cu at (211.5, 99.0)
- added R17: 1k5, Resistor_SMD:R_0402_1005Metric, F.Cu at (124.5, 83.5)
- added R18: 100R, Resistor_SMD:R_0402_1005Metric, F.Cu at (126.5, 83.5)
- added R19: 100R, Resistor_SMD:R_0402_1005Metric, F.Cu at (128.5, 83.5)
- added R2: 4k7, Resistor_SMD:R_0402_1005Metric, F.Cu at (210.0, 85.0)
- added R20: 1k5, Resistor_SMD:R_0402_1005Metric, F.Cu at (130.5, 83.5)
- added R21: 1k5, Resistor_SMD:R_0402_1005Metric, F.Cu at (132.5, 83.5)
- added R22: 50R, Resistor_SMD:R_0402_1005Metric, F.Cu at (155.5, 78.0)
- added R23: 1k5, Resistor_SMD:R_0402_1005Metric, F.Cu at (123.5, 90.0)
- added R24: 82k, Resistor_SMD:R_0402_1005Metric, F.Cu at (120.0, 98.5)
- added R25: 1k5, Resistor_SMD:R_0402_1005Metric, F.Cu at (119.3, 102.4)
- added R26: 10k, Resistor_SMD:R_0402_1005Metric, F.Cu at (181.0, 99.0)
- added R27: 4k7, Resistor_SMD:R_0402_1005Metric, F.Cu at (201.5, 129.5)
- added R28: 10R, Resistor_SMD:R_0603_1608Metric, F.Cu at (118.7, 146.5)
- added R29: 91k, Resistor_SMD:R_0402_1005Metric, F.Cu at (112.0, 140.0)
- added R3: 10R, Resistor_SMD:R_0402_1005Metric, F.Cu at (112.0, 81.5)
- added R30: 4k7, Resistor_SMD:R_0402_1005Metric, F.Cu at (111.0, 140.0)
- added R31: 100k, Resistor_SMD:R_0402_1005Metric, F.Cu at (115.0, 138.5)
- added R32: 33k, Resistor_SMD:R_0402_1005Metric, F.Cu at (104.5, 119.0)
- added R33: 4k7, Resistor_SMD:R_0402_1005Metric, F.Cu at (141.0, 81.0)
- added R34: 12k, Resistor_SMD:R_0402_1005Metric, F.Cu at (101.5, 115.5)
- added R35: 3k9, Resistor_SMD:R_0402_1005Metric, F.Cu at (101.5, 118.0)
- added R36: 100R, Resistor_SMD:R_0402_1005Metric, F.Cu at (196.0, 101.0)
- added R37: 100R, Resistor_SMD:R_0402_1005Metric, F.Cu at (195.0, 101.0)
- added R38: 100R, Resistor_SMD:R_0402_1005Metric, F.Cu at (181.5, 120.0)
- added R39: R, Resistor_SMD:R_0603_1608Metric, F.Cu at (190.0, 100.7)
- added R4: 5k1, Resistor_SMD:R_0402_1005Metric, F.Cu at (112.0, 82.5)
- added R42: 10R, Resistor_SMD:R_0402_1005Metric, F.Cu at (184.0, 119.0)
- added R43: R, Resistor_SMD:R_0805_2012Metric, F.Cu at (200.0, 107.6)
- added R44: R, Resistor_SMD:R_0805_2012Metric, F.Cu at (194.5, 119.5)
- added R45: R, Resistor_SMD:R_0805_2012Metric, F.Cu at (189.5, 119.6)
- added R46: 39k, Resistor_SMD:R_0402_1005Metric, F.Cu at (194.0, 123.0)
- added R47: 39k, Resistor_SMD:R_0402_1005Metric, F.Cu at (189.0, 123.0)
- added R48: 82k, Resistor_SMD:R_0402_1005Metric, F.Cu at (199.0, 122.5)
- added R49: 1k5, Resistor_SMD:R_0402_1005Metric, F.Cu at (201.5, 122.5)
- added R5: 5k1, Resistor_SMD:R_0402_1005Metric, F.Cu at (112.0, 85.5)
- added R50: 100R, Resistor_SMD:R_0402_1005Metric, F.Cu at (167.5, 104.0)
- added R51: 100R, Resistor_SMD:R_0402_1005Metric, F.Cu at (166.5, 104.0)
- added R52: 100R, Resistor_SMD:R_0402_1005Metric, F.Cu at (153.0, 120.0)
- added R53: R, Resistor_SMD:R_0603_1608Metric, F.Cu at (160.5, 103.2)
- added R56: 10R, Resistor_SMD:R_0402_1005Metric, F.Cu at (155.0, 120.0)
- added R57: R, Resistor_SMD:R_0805_2012Metric, F.Cu at (171.0, 111.6)
- added R58: R, Resistor_SMD:R_0805_2012Metric, F.Cu at (166.0, 121.6)
- added R59: R, Resistor_SMD:R_0805_2012Metric, F.Cu at (159.5, 121.4)
- added R6: 1k5, Resistor_SMD:R_0402_1005Metric, F.Cu at (210.0, 83.5)
- added R60: 39k, Resistor_SMD:R_0402_1005Metric, F.Cu at (164.0, 127.0)
- added R61: 39k, Resistor_SMD:R_0402_1005Metric, F.Cu at (159.0, 127.0)
- added R62: 82k, Resistor_SMD:R_0402_1005Metric, F.Cu at (171.0, 123.0)
- added R63: 1k5, Resistor_SMD:R_0402_1005Metric, F.Cu at (171.0, 125.0)
- added R64: 100R, Resistor_SMD:R_0402_1005Metric, F.Cu at (140.5, 104.5)
- added R65: 100R, Resistor_SMD:R_0402_1005Metric, F.Cu at (139.5, 104.5)
- added R66: 100R, Resistor_SMD:R_0402_1005Metric, F.Cu at (127.0, 121.0)
- added R67: R, Resistor_SMD:R_0603_1608Metric, F.Cu at (133.0, 103.7)
- added R7: 22R, Resistor_SMD:R_0402_1005Metric, F.Cu at (112.0, 83.5)
- added R70: 10R, Resistor_SMD:R_0402_1005Metric, F.Cu at (129.0, 121.0)
- added R71: R, Resistor_SMD:R_0805_2012Metric, F.Cu at (144.5, 112.1)
- added R72: R, Resistor_SMD:R_0805_2012Metric, F.Cu at (139.5, 123.0)
- added R73: R, Resistor_SMD:R_0805_2012Metric, F.Cu at (133.0, 123.0)
- added R74: 39k, Resistor_SMD:R_0402_1005Metric, F.Cu at (138.5, 126.5)
- added R75: 39k, Resistor_SMD:R_0402_1005Metric, F.Cu at (133.5, 126.5)
- added R76: 82k, Resistor_SMD:R_0402_1005Metric, F.Cu at (143.0, 126.5)
- added R77: 1k5, Resistor_SMD:R_0402_1005Metric, F.Cu at (145.5, 127.5)
- added R8: 22R, Resistor_SMD:R_0402_1005Metric, F.Cu at (112.0, 84.5)
- added R9: 1k5, Resistor_SMD:R_0402_1005Metric, F.Cu at (115.0, 85.0)
- added TP1: TestPoint, TestPoint:TestPoint_Pad_D1.5mm, F.Cu at (166.0, 94.0)
- added TP10: TestPoint, TestPoint:TestPoint_Pad_D1.5mm, F.Cu at (112.0, 98.0)
- added TP2: TestPoint, TestPoint:TestPoint_Pad_D1.5mm, F.Cu at (116.5, 99.0)
- added TP3: TestPoint, TestPoint:TestPoint_Pad_D1.5mm, F.Cu at (156.0, 87.5)
- added TP4: TestPoint, TestPoint:TestPoint_Pad_D1.5mm, F.Cu at (161.5, 93.0)
- added TP5: TestPoint, TestPoint:TestPoint_Pad_D1.5mm, F.Cu at (177.5, 103.0)
- added TP6: TestPoint, TestPoint:TestPoint_Pad_D1.5mm, F.Cu at (178.5, 94.0)
- added TP7: TestPoint, TestPoint:TestPoint_Pad_D1.5mm, F.Cu at (122.5, 146.5)
- added TP8: TestPoint, TestPoint:TestPoint_Pad_D1.5mm, F.Cu at (143.5, 83.5)
- added TP9: TestPoint, TestPoint:TestPoint_Pad_D1.5mm, F.Cu at (117.5, 98.0)
- added U1: STM32F303CBTx, Package_QFP:LQFP-48_7x7mm_P0.5mm, F.Cu at (163.5, 82.5)
- added U2: LM5017MR, Package_SO:SOIC-8-1EP_3.9x4.9mm_P1.27mm_EP2.95x4.9mm_Mask2.71x3.4mm_ThermalVias, F.Cu at (113.0, 133.5)
- added U3: TPS76333, Package_TO_SOT_SMD:SOT-23-5, F.Cu at (139.0, 87.5)
- added U4: INA240A1PW, Package_SO:TSSOP-8_4.4x3mm_P0.65mm, F.Cu at (184.5, 125.5)
- added U5: UCC21520DW, Package_SO:SOIC-16W_7.5x10.3mm_P1.27mm, F.Cu at (191.5, 109.0)
- added U6: INA240A1PW, Package_SO:TSSOP-8_4.4x3mm_P0.65mm, F.Cu at (153.9, 125.7)
- added U7: UCC21520DW, Package_SO:SOIC-16W_7.5x10.3mm_P1.27mm, F.Cu at (162.8, 111.3)
- added U8: INA240A1PW, Package_SO:TSSOP-8_4.4x3mm_P0.65mm, F.Cu at (128.0, 126.5)
- added U9: UCC21520DW, Package_SO:SOIC-16W_7.5x10.3mm_P1.27mm, F.Cu at (136.1, 112.0)
- added Y1: ASE-8.000MHZ-LC-T, Oscillator:Oscillator_SMD_Abracon_ASE-4Pin_3.2x2.5mm, F.Cu at (152.0, 79.0)
Other:
- board outline added: 120 x 75 mm
